Commit message: edit

File: description/robot_core.xacro (robot description, xacro)
@@ -5,5 +5,5 @@
     <xacro:property name="chassis_width" value="0.19"/>
     <xacro:property name="chassis_height" value="0.17"/>
-    <xacro:property name="chassis_mass" value="1.0"/>
+    <xacro:property name="chassis_mass" value="3.0"/>
     <xacro:property name="wheel_radius" value="0.034"/>
     <xacro:property name="wheel_thickness" value="0.027"/>
@@ -13,5 +13,5 @@
     <xacro:property name="wheel_offset_z" value="-0.016"/>
     <xacro:property name="caster_wheel_radius" value="0.024"/>
-    <xacro:property name="caster_wheel_mass" value="0.01"/>
+    <xacro:property name="caster_wheel_mass" value="0.5"/>
     <xacro:property name="caster_wheel_offset_x" value="0.035"/>
     <xacro:property name="caster_wheel_offset_z" value="${wheel_offset_z - wheel_radius + caster_wheel_radius}"/>
@@ -145,6 +145,6 @@
     <gazebo reference="caster_wheel">
         <material>Gazebo/Red</material>
-        <mu1 value="0.001"/>
-        <mu2 value="0.001"/>
+        <mu1 value="0.01"/>
+        <mu2 value="0.01"/>
     </gazebo>
 </robot>
